File: passive-lipo-balancer-nano.kicad_sch (KiCad schematic)
At the start: 31 parts, among them J1 Conn_01x04, J2 Conn_01x04, Q1 MTN2306AN3, Q2 MTN2306AN3, Q3 MTN2306AN3, SW1 SW_DIP_x01, U1 ER_OLEDM0.91_1x-I2C

Commit message: code arduino sketch sch fix
Parts:
- removed R1, R2: 4k7Ω, symbol Device:R
- renumbered R3 to R1, R12 to R10, R13 to R11, R14 to R12, R15 to R13, R16 to R14, R17 to R15, R4 to R2, R5 to R3, R6 to R4, R7 to R5, R8 to R6, R9 to R7, R10 to R8, R11 to R9
Other:
- note removed: "I2Cバスのプルアップ抵抗"

Commit message: fix sketch fix sch
Parts:
- added C7: Cell2, symbol Device:C
- added C8: Cell1, symbol Device:C
- added J2, J4: Conn_01x03, Connector_JST:JST_XH_S3B-XH-A_1x03_P2.50mm_Horizontal, symbol Connector_Generic:Conn_01x03
- renumbered J2 to J3, R3 to R1, R4 to R2, R1 to R3, R2 to R4, R6 to R5, R7 to R6, R5 to R7
Connections:
- net GND: now also J1.4 (Pin_4), J2.3 (Pin_3)
- net Cell1+: now reaches R1.1
- net Cell1+: now also J1.3 (Pin_3), R7.2, J2.2 (Pin_2); no longer J1.1 (Pin_1)
- removed net Cell1-: J1.4 (Pin_4), R7.2
- removed net Cell2-: J1.3 (Pin_3), R12.2, R8.1
- net Cell3- renamed Cell2+
- net Cell2+: now also R12.2, J2.1 (Pin_1); no longer R15.2
- new net: C7.2, C8.1, J4.2 (Pin_2)
- new net: C8.2, J4.3 (Pin_3)
- new net: C7.1, J4.1 (Pin_1)
- new net Cell3+: J1.1 (Pin_1), R15.2, R8.1
Other:
- note added: "ストレージモード/バランスモード"
- note removed: "ストレージモード（すべてのセルを3.8Vまで放電）と バランスモード（一番電圧の低いセルと同じ電圧まで放電）の切り替え"
- moved on the sheet: R1, R2, R5, R6, R8, R9

Commit message: add JP1(BT Cell2+ to Nano VIN)
Parts:
- added JP1: Jumper_2_Open, Package_LCC:PLCC-84_29.3x29.3mm_P1.27mm, symbol Jumper:Jumper_2_Open
Connections:
- net Cell2+: now also JP1.1 (A)
- net at A1.30 (VIN): now also JP1.2 (B)
- no-connect marks 18 -> 17
Other:
- note added: "JP1をショートして バッテリーから給電すると USB給電なしで動作可能に"
Changed lines of the file:
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@@
 		)
 	)
+	(text "JP1をショートして\nバッテリーから給電すると\nUSB給電なしで動作可能に"
+		(exclude_from_sim no)
+		(at 58.166 16.51 0)
+		(effects
+			(font
+				(size 1.27 1.27)
+			)
+		)
+	)
 	(text_box "ストレージモード：すべてのセルを3.8Vまで放電\nバランスモード：一番電圧の低いセルと同じ電圧まで放電"
 		(exclude_from_sim no)
@@
 	)
 	(junction
+		(at 73.66 26.67)
+		(diameter 0)
+		(color 0 0 0 0)
+	)
+	(junction
 		(at 152.4 152.4)
 		(diameter 0)
@@
 	)
 	(no_connect
-		(at 73.66 27.94)
-	)
-	(no_connect
 		(at 63.5 63.5)
 	)
@@
 	(wire
 		(pts
+			(xy 73.66 25.4) (xy 73.66 27.94)
+		)
+		(stroke
+			(width 0)
+			(type default)
+		)
+	)
+	(wire
+		(pts
 			(xy 194.31 135.89) (xy 198.12 135.89)
 		)
@@
 	(wire
 		(pts
+			(xy 50.8 26.67) (xy 53.34 26.67)
+		)
+		(stroke
+			(width 0)
+			(type default)
+		)
+	)
+	(wire
+		(pts
 			(xy 209.55 152.4) (xy 198.12 152.4)
 		)
@@
 	(wire
 		(pts
+			(xy 73.66 26.67) (xy 63.5 26.67)
+		)
+		(stroke
+			(width 0)
+			(type default)
+		)
+	)
+	(wire
+		(pts
 			(xy 254 152.4) (xy 254 148.59)
 		)
@@
 		)
 	)
+	(global_label "Cell2+"
+		(shape input)
+		(at 50.8 26.67 180)
+		(fields_autoplaced yes)
+		(effects
+			(font
+				(size 1.27 1.27)
+			)
+			(justify right)
+		)
+		(property "Intersheetrefs" "${INTERSHEET_REFS}"
+			(at 41.3439 26.67 0)
+			(hide yes)
+			(show_name no)
+			(do_not_autoplace no)
+			(effects
+				(font
+					(size 1.27 1.27)
+				)
+				(justify right)
+			)
+		)
+	)
 	(global_label "SDA"
 		(shape bidirectional)
@@
 	)
 	(symbol
+		(lib_id "Jumper:Jumper_2_Open")
+		(at 58.42 26.67 0)
+		(unit 1)
+		(body_style 1)
+		(exclude_from_sim no)
+		(in_bom yes)
+		(on_board yes)
+		(in_pos_files yes)
+		(dnp no)
+		(fields_autoplaced yes)
+		(property "Reference" "JP1"
+			(at 58.42 20.32 0)
+			(show_name no)
+			(do_not_autoplace no)
+			(effects
+				(font
+					(size 1.27 1.27)
+				)
+			)
+		)
+		(property "Value" "Jumper_2_Open"
+			(at 58.42 22.86 0)
+			(show_name no)
+			(do_not_autoplace no)
+			(effects
+				(font
+					(size 1.27 1.27)
+				)
+			)
+		)
+		(property "Footprint" "Package_LCC:PLCC-84_29.3x29.3mm_P1.27mm"
+			(at 58.42 26.67 0)
+			(hide yes)
+			(show_name no)
+			(do_not_autoplace no)
+			(effects
+				(font
+					(size 1.27 1.27)
+				)
+			)
+		)
+		(property "Datasheet" ""
+			(at 58.42 26.67 0)
+			(hide yes)
+			(show_name no)
+			(do_not_autoplace no)
+			(effects
+				(font
+					(size 1.27 1.27)
+				)
+			)
+		)
+		(property "Description" "Jumper, 2-pole, open"
+			(at 58.42 26.67 0)
+			(hide yes)
+			(show_name no)
+			(do_not_autoplace no)
+			(effects
+				(font
+					(size 1.27 1.27)
+				)
+			)
+		)
+		(pin "2"
+		)
+		(pin "1"
+		)
+		(instances
+			(project "passive-lipo-balancer-nano"
+				(path "/72d8573a-db7d-420b-a0f0-68b69316f634"
+					(reference "JP1")
+					(unit 1)
+				)
+			)
+		)
+	)
+	(symbol
 		(lib_id "Device:R")
 		(at 128.27 44.45 0)
@@
 					(unit 1)
 				)
+			)
+		)
+	)
+	(symbol
+		(lib_id "power:PWR_FLAG")
+		(at 73.66 25.4 0)
+		(unit 1)
+		(body_style 1)
+		(exclude_from_sim no)
+		(in_bom yes)
+		(on_board yes)
+		(in_pos_files yes)
+		(dnp no)
+		(fields_autoplaced yes)
+		(property "Reference" "#FLG02"
+			(at 73.66 23.495 0)
+			(hide yes)
+			(show_name no)
+			(do_not_autoplace no)
+			(effects
+				(font
+					(size 1.27 1.27)
+				)
+			)
+		)
+		(property "Value" "PWR_FLAG"
+			(at 73.66 20.32 0)
+			(show_name no)
+			(do_not_autoplace no)
+			(effects
+				(font
+					(size 1.27 1.27)
+				)
+			)
+		)
+		(property "Footprint" ""
+			(at 73.66 25.4 0)
+			(hide yes)
+			(show_name no)
+			(do_not_autoplace no)
+			(effects
+				(font
+					(size 1.27 1.27)
+				)
+			)
+		)
+		(property "Datasheet" ""
+			(at 73.66 25.4 0)
+			(hide yes)
+			(show_name no)
+			(do_not_autoplace no)
+			(effects
+				(font
+					(size 1.27 1.27)
+				)
+			)
+		)
+		(property "Description" "Special symbol for telling ERC where power comes from"
+			(at 73.66 25.4 0)
+			(hide yes)
+			(show_name no)
+			(do_not_autoplace no)
+			(effects
+				(font
+					(size 1.27 1.27)
+				)
+			)
+		)
+		(pin "1"
+		)
+		(instances
+			(project "passive-lipo-balancer-nano"
+				(path "/72d8573a-db7d-420b-a0f0-68b69316f634"
+					(reference "#FLG02")
+					(unit 1)
+				)

Commit message: apply footprint
Parts:
- JP1: footprint Package_LCC:PLCC-84_29.3x29.3mm_P1.27mm -> Connector_PinHeader_2.54mm:PinHeader_1x02_P2.54mm_Vertical
- R1, R7: footprint (none) -> Resistor_THT:R_Axial_DIN0207_L6.3mm_D2.5mm_P10.16mm_Horizontal
- R10: renamed from R3; footprint (none) -> Resistor_THT:R_Axial_DIN0207_L6.3mm_D2.5mm_P10.16mm_Horizontal
- R11: renamed from R10; footprint (none) -> Resistor_THT:R_Axial_DIN0207_L6.3mm_D2.5mm_P10.16mm_Horizontal
- R12: renamed from R13; footprint (none) -> Resistor_THT:R_Axial_DIN0207_L6.3mm_D2.5mm_P10.16mm_Horizontal
- R13: renamed from R4; value 10kΩ -> 100kΩ; footprint (none) -> Resistor_THT:R_Axial_DIN0207_L6.3mm_D2.5mm_P10.16mm_Horizontal
- R14: renamed from R11; value 10kΩ -> 100kΩ; footprint (none) -> Resistor_THT:R_Axial_DIN0207_L6.3mm_D2.5mm_P10.16mm_Horizontal
- R15: renamed from R14; value 10kΩ -> 100kΩ; footprint (none) -> Resistor_THT:R_Axial_DIN0207_L6.3mm_D2.5mm_P10.16mm_Horizontal
- R2: renamed from R5; footprint (none) -> Resistor_THT:R_Axial_DIN0207_L6.3mm_D2.5mm_P10.16mm_Horizontal
- R3: renamed from R8; footprint (none) -> Resistor_THT:R_Axial_DIN0207_L6.3mm_D2.5mm_P10.16mm_Horizontal
- R4: renamed from R2; footprint (none) -> Resistor_THT:R_Axial_DIN0207_L6.3mm_D2.5mm_P10.16mm_Horizontal
- R5: renamed from R6; footprint (none) -> Resistor_THT:R_Axial_DIN0207_L6.3mm_D2.5mm_P10.16mm_Horizontal
- R6: renamed from R9; footprint (none) -> Resistor_THT:R_Axial_DIN0207_L6.3mm_D2.5mm_P10.16mm_Horizontal
- R8: renamed from R12; footprint (none) -> Resistor_THT:R_Axial_DIN0207_L6.3mm_D2.5mm_P10.16mm_Horizontal
- R9: renamed from R15; footprint (none) -> Resistor_THT:R_Axial_DIN0207_L6.3mm_D2.5mm_P10.16mm_Horizontal
- renumbered C7 to C4, C8 to C5, C4 to C6, C5 to C7, C6 to C8, J2 to J1, J1 to J2, J4 to J3, J3 to J4
Other:
- moved on the sheet: J1, J2, J3, J4

Commit message: fix oled footprint
Parts:
- C1, C2, C3: footprint (none) -> Capacitor_THT:C_Disc_D5.0mm_W2.5mm_P2.50mm
- SW1: footprint Button_Switch_SMD:Nidec_Copal_CAS-120A -> Button_Switch_THT:SW_DIP_SPSTx01_Slide_9.78x4.72mm_W7.62mm_P2.54mm
Changed lines of the file:
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@@
 	(title_block
 		(date "2026-10-27")
+		(rev "${REVISION}")
 	)
 	(text "D13はNanoのオンボードLED\nとつながっている\n放電中は光らせる？"
@@
 			)
 		)
-		(property "Footprint" ""
+		(property "Footprint" "Capacitor_THT:C_Disc_D5.0mm_W2.5mm_P2.50mm"
 			(at 35.2552 119.38 0)
 			(hide yes)
@@
 			)
 		)
-		(property "Footprint" ""
+		(property "Footprint" "Capacitor_THT:C_Disc_D5.0mm_W2.5mm_P2.50mm"
 			(at 47.9552 119.38 0)
 			(hide yes)
@@
 			)
 		)
-		(property "Footprint" "Button_Switch_SMD:Nidec_Copal_CAS-120A"
+		(property "Footprint" "Button_Switch_THT:SW_DIP_SPSTx01_Slide_9.78x4.72mm_W7.62mm_P2.54mm"
 			(at 34.29 58.42 0)
 			(hide yes)
@@
 			)
 		)
-		(property "Footprint" ""
+		(property "Footprint" "Capacitor_THT:C_Disc_D5.0mm_W2.5mm_P2.50mm"
 			(at 22.5552 119.38 0)
 			(hide yes)
